File: motoVindicator.kicad_pcb (KiCad board)
At the start: 2 copper layers, 53.3 x 19 mm, 13 parts, among them J1 J1, J3 Conn_01x02_Male, U1 4N37, U2 4N37

Commit message: R3 and R6 adjusted
Parts:
- J1: value J1 -> Conn_01x04_Male
- R3: value 24.5k -> 26k
- R6: value 19.8k -> 20k
